File: ist_project/ist_project.kicad_pcb (KiCad board)
At the start: 2 copper layers, 38 parts, among them J1 Conn_01x04, J10 Conn_01x04, J11 Conn_01x04, J12 Conn_01x04, J13 Conn_01x04, J2 Conn_01x04, J3 Conn_01x04, J4 Conn_01x04, J5 Conn_01x04, J6 Conn_01x04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

Commit message: 회로도 수정 / pcb 작업중
Parts:
- removed J1, J10, J11, J12, J13, J2, J3, J4, J5, J6, J7, J8, J9: Conn_01x04, Connector_Molex:Molex_SPOX_5267-04A_1x04_P2.50mm_Vertical
- added J_BTN_1: Conn_01x04, Connector_Molex:Molex_SPOX_5267-04A_1x04_P2.50mm_Vertical, F.Cu at (49.5, 55.9)
- added J_BTN_2: Conn_01x04, Connector_Molex:Molex_SPOX_5267-04A_1x04_P2.50mm_Vertical, F.Cu at (49.5, 66.0)
- added J_BTN_3: Conn_01x04, Connector_Molex:Molex_SPOX_5267-04A_1x04_P2.50mm_Vertical, F.Cu at (49.5, 76.2)
- added J_BTN_4: Conn_01x04, Connector_Molex:Molex_SPOX_5267-04A_1x04_P2.50mm_Vertical, F.Cu at (49.5, 86.4)
- added J_BTN_5: Conn_01x04, Connector_Molex:Molex_SPOX_5267-04A_1x04_P2.50mm_Vertical, F.Cu at (49.5, 96.5)
- added J_BTN_6: Conn_01x04, Connector_Molex:Molex_SPOX_5267-04A_1x04_P2.50mm_Vertical, F.Cu at (49.5, 106.7)
- added J_BTN_7: Conn_01x04, Connector_Molex:Molex_SPOX_5267-04A_1x04_P2.50mm_Vertical, F.Cu at (49.5, 116.8)
- added J_BTN_EFFECT0: Conn_01x04, Connector_Molex:Molex_SPOX_5267-04A_1x04_P2.50mm_Vertical, F.Cu at (93.0, 55.9)
- added J_BTN_START0: Conn_01x04, Connector_Molex:Molex_SPOX_5267-04A_1x04_P2.50mm_Vertical, F.Cu at (93.0, 66.0)
- added J_BTN_VEFX0: Conn_01x04, Connector_Molex:Molex_SPOX_5267-04A_1x04_P2.50mm_Vertical, F.Cu at (93.0, 76.2)
- added J_BT_Conn0: Conn_01x04, Connector_Molex:Molex_SPOX_5267-04A_1x04_P2.50mm_Vertical, F.Cu at (71.2, 116.8)
- added J_TURN_Conn0: Conn_01x04, Connector_Molex:Molex_SPOX_5267-04A_1x04_P2.50mm_Vertical, F.Cu at (93.0, 86.3)
- added J_USB_Conn0: Conn_01x04, Connector_Molex:Molex_SPOX_5267-04A_1x04_P2.50mm_Vertical, F.Cu at (71.2, 55.9)
- moved R8 76.1 mm to (61.2, 59.9)
- moved R9 71.7 mm to (61.2, 70.1)
- moved R10 67.8 mm to (61.2, 80.3)
- moved R2 65.6 mm to (65.5, 62.5), turned to -90 degrees
- moved R11 64.5 mm to (61.2, 90.4)
- moved R12 63.6 mm to (61.2, 100.6)
- moved R13 63.4 mm to (61.2, 111.0)
- moved R14 62.5 mm to (62.2, 115.8)
- moved R1 60.2 mm to (65.5, 68.3), turned to -90 degrees
- moved C1 55.2 mm to (65.3, 48.5), turned to 90 degrees
- moved R4 54.2 mm to (84.6, 66.5)
- moved C2 52.3 mm to (70.2, 48.5), turned to 90 degrees
- moved SW1 50.4 mm to (75.0, 104.1)
- moved U1 50.2 mm to (75.0, 71.1)
- moved Y1 50.0 mm to (75.0, 85.7)
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Routing:
- net VCC: track 0.00 -> 355.2 mm
- net GND: track 0.00 -> 32.3 mm, vias 0 -> 4
- net Net-(U1-XTAL1): track 0.00 -> 16.8 mm
- net Net-(U1-XTAL2): track 0.00 -> 16.5 mm
- net /BT_7: track 0.00 -> 13.2 mm
- net Net-(U1-~{RESET}): track 0.00 -> 11.6 mm
- net /BT_6: track 0.00 -> 10.7 mm
- net /BT_START: track 0.00 -> 10.6 mm
- net /BT_VEFX: track 0.00 -> 10.6 mm
- net /BT_EFFECT: track 0.00 -> 10.5 mm
- net /BT_1: track 0.00 -> 10.4 mm
- net /BT_2: track 0.00 -> 10.4 mm
- net /BT_4: track 0.00 -> 10.4 mm
- net /BT_5: track 0.00 -> 10.4 mm
- net /BT_3: track 0.00 -> 10.4 mm
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
Commit message: PCB 그리기 완료 / Mount Hole 추가
Parts:
- added H1: MountingHole, MountingHole:MountingHole_3.2mm_M3_ISO7380_Pad_TopOnly, F.Cu at (43.7, 47.5)
- added H2: MountingHole, MountingHole:MountingHole_3.2mm_M3_ISO7380_Pad_TopOnly, F.Cu at (108.0, 47.5)
- added H3: MountingHole, MountingHole:MountingHole_3.2mm_M3_ISO7380_Pad_TopOnly, F.Cu at (43.7, 122.9)
- added H4: MountingHole, MountingHole:MountingHole_3.2mm_M3_ISO7380_Pad_TopOnly, F.Cu at (108.0, 122.9)
- renumbered J_TURN_Conn0 to J_TURNTABLE_Conn0
Routing:
- net /BT_7: track 13.2 -> 83.0 mm, vias 0 -> 8
- net /BT_6: track 10.7 -> 73.6 mm, vias 0 -> 8
- net /TXD1_BT: track 0.00 -> 54.6 mm, vias 0 -> 4
- net /BT_4: track 10.4 -> 64.3 mm, vias 0 -> 8
- net /RXD1_BT: track 0.00 -> 51.4 mm, vias 0 -> 2
- net /BT_VEFX: track 10.6 -> 61.9 mm, vias 0 -> 6
- net Net-(U1-~{RESET}): track 11.6 -> 56.2 mm, vias 0 -> 2
- net /BT_START: track 10.6 -> 53.6 mm, vias 0 -> 3
- net /BT_EFFECT: track 10.5 -> 52.9 mm, vias 0 -> 3
- net /BT_3: track 10.4 -> 51.8 mm, vias 0 -> 4
- net /SC_1: track 0.00 -> 37.1 mm, vias 0 -> 8
- net /SC_0: track 0.00 -> 36.7 mm, vias 0 -> 8
- net /BT_5: track 10.4 -> 41.6 mm, vias 0 -> 2
- net /BT_2: track 10.4 -> 35.2 mm, vias 0 -> 2
- net /BT_1: track 10.4 -> 30.6 mm
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- added copper zone on B.Cu, net GND
- added copper zone on F.Cu, net GND
Other:
- board outline added: 74.4 x 85.1 mm
